File: Hardware/TMR01/TMR01.sch (EAGLE design)
At the start: 38 parts, among them U1 ATMEGA328P_TQFP, U2 DS3234

Commit message: Board created with a watch layout
Parts:
- J1: device SparkFun-Connectors:6_PIN_SERIAL_TARGET -> SparkFun-Connectors:CONN_06SMD-FEMALE-V2
- J2: device SparkFun-Connectors:CONN_04 -> SparkFun-Connectors:CONN_06SMD-FEMALE-V2
Connections:
- removed net N$10: R2.2
- removed net N$11: R3.2
- removed net N$12: R4.2
- removed net N$13: R5.2
- removed net N$14: R6.2
- removed net N$15: R7.2
- removed net N$16: R8.2
- removed net N$19: R9.2
- removed net N$21: R10.2
- removed net N$23: R11.2
- removed net N$25: R12.2
- removed net N$26: R15.2, U2.INT/SQW
- removed net N$28: U1.PB2(SS/OC1B)
- removed net N$29: U1.PB1(OC1A)
- removed net N$30: U1.PB0(ICP)
- removed net N$33: U1.PD2(INT0)
- removed net N$34: U1.PD3(INT1)
- removed net N$35: U1.PD4(XCK/T0)
- removed net N$36: U1.PD5(T1)
- removed net N$37: U1.PD6(AIN0)
- removed net N$38: U1.PD7(AIN1)
- removed net N$40: U2.CS
- removed net N$9: R1.2
- new net D1: R11.2, U1.PD2(INT0)
- new net D10: R2.2, U1.PC1(ADC1)
- new net D11: R1.2, U1.PC2(ADC2)
- new net D12: R12.2, U1.PC3(ADC3)
- new net D2: R10.2, U1.PD3(INT1)
- new net D3: R9.2, U1.PD4(XCK/T0)
- new net D4: R8.2, U1.PD5(T1)
- new net D5: R7.2, U1.PD6(AIN0)
- new net D6: R6.2, U1.PD7(AIN1)
- new net D7: R5.2, U1.PB0(ICP)
- new net D8: R4.2, U1.PB1(OC1A)
- new net D9: R3.2, U1.PC0(ADC0)
- new net SQW: J2.1, R15.2, U2.INT/SQW
- new net SS: J2.2, U1.PB2(SS/OC1B), U2.CS
- net DTR: now also J1.1; no longer J1.DTR
- net GND: now also J1.5, J1.6; no longer J1.CTS, J1.GND
- net MISO: now also J2.5; no longer J2.3
- net MOSI: now also J2.4; no longer J2.2
- net PUSH: now also U1.PC4(ADC4/SDA)
- net RST: now also J2.3; no longer J2.1
- net RX: now also J1.3; no longer J1.TXO
- net SCK: now also J2.6; no longer J2.4
- net TX: now also J1.2; no longer J1.RXI
- net VCC: now also J1.4; no longer J1.VCC
Other:
- note added: "Alejandro Herrero"
- moved on the sheet: BT1, C3, J1, R14, S1

Commit message: connecting grounds and vcc with via
Parts:
- removed C4: 22pF, Perfect_0402:CAP_0402
Connections:
- net GND: no longer C4.2
- net VCC: no longer C4.1
Changed lines of the file:
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@@
 <part name="SUPPLY5" library="SparkFun-PowerSymbols" deviceset="VCC" device=""/>
 <part name="R15" library="SparkFun-Resistors" deviceset="RESISTOR" device="0402" value="10k"/>
-<part name="C4" library="Perfect_0402" deviceset="CAP_0402" device="" value="22pF"/>
-<part name="GND6" library="SparkFun-PowerSymbols" deviceset="GND" device=""/>
 <part name="J1" library="SparkFun-Connectors" deviceset="CONN_06" device="SMD-FEMALE-V2"/>
 <part name="J2" library="SparkFun-Connectors" deviceset="CONN_06" device="SMD-FEMALE-V2"/>
@@
 <attribute name="NAME" x="180.34" y="57.404" size="1.778" layer="95" font="vector" align="bottom-center"/>
 <attribute name="VALUE" x="180.34" y="54.356" size="1.778" layer="96" font="vector" align="top-center"/>
-</instance>
-<instance part="C4" gate="G$1" x="170.18" y="45.72">
-<attribute name="NAME" x="171.704" y="51.181" size="1.778" layer="95"/>
-<attribute name="VALUE" x="171.704" y="46.101" size="1.778" layer="96"/>
-</instance>
-<instance part="GND6" gate="1" x="170.18" y="40.64">
-<attribute name="VALUE" x="170.18" y="40.386" size="1.778" layer="96" align="top-center"/>
 </instance>
 <instance part="J1" gate="G$1" x="81.28" y="154.94">
@@
 <junction x="226.06" y="68.58"/>
 </segment>
-<segment>
-<pinref part="GND6" gate="1" pin="GND"/>
-<pinref part="C4" gate="G$1" pin="2"/>
-<wire x1="170.18" y1="43.18" x2="170.18" y2="45.72" width="0.1524" layer="91"/>
-</segment>
 </net>
 <net name="VCC" class="0">
@@
 <wire x1="190.5" y1="76.2" x2="185.42" y2="76.2" width="0.1524" layer="91"/>
 <wire x1="185.42" y1="76.2" x2="185.42" y2="81.28" width="0.1524" layer="91"/>
+<wire x1="170.18" y1="76.2" x2="185.42" y2="76.2" width="0.1524" layer="91"/>
+<junction x="185.42" y="76.2"/>
 <pinref part="R15" gate="G$1" pin="1"/>
 <wire x1="175.26" y1="55.88" x2="170.18" y2="55.88" width="0.1524" layer="91"/>
 <wire x1="170.18" y1="55.88" x2="170.18" y2="76.2" width="0.1524" layer="91"/>
-<wire x1="170.18" y1="76.2" x2="185.42" y2="76.2" width="0.1524" layer="91"/>
-<junction x="185.42" y="76.2"/>
-<pinref part="C4" gate="G$1" pin="1"/>
-<wire x1="170.18" y1="53.34" x2="170.18" y2="55.88" width="0.1524" layer="91"/>
-<junction x="170.18" y="55.88"/>
-</segment>
-<segment>
+</segment>
+<segment>

Commit message: everything except D7
Parts:
- removed R15: 10k, SparkFun-Resistors:RESISTOR0402
- J2: device SparkFun-Connectors:CONN_06SMD-FEMALE-V2 -> SparkFun-Connectors:CONN_04SMD_RA_FEMALE
Connections:
- removed net SQW: J2.1, R15.2, U2.INT/SQW
- net MISO: now also J2.3; no longer J2.5
- net MOSI: now also J2.2; no longer J2.4
- net RST: now also J2.1; no longer J2.3
- net SCK: now also J2.4; no longer J2.6
- net SS: no longer J2.2
- net VCC: no longer R15.1
Changed lines of the file:
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@@
 <part name="SUPPLY4" library="SparkFun-PowerSymbols" deviceset="VCC" device=""/>
 <part name="SUPPLY5" library="SparkFun-PowerSymbols" deviceset="VCC" device=""/>
-<part name="R15" library="SparkFun-Resistors" deviceset="RESISTOR" device="0402" value="10k"/>
 <part name="J1" library="SparkFun-Connectors" deviceset="CONN_06" device="SMD-FEMALE-V2"/>
-<part name="J2" library="SparkFun-Connectors" deviceset="CONN_06" device="SMD-FEMALE-V2"/>
+<part name="J2" library="SparkFun-Connectors" deviceset="CONN_04" device="SMD_RA_FEMALE"/>
 </parts>
 <sheets>
@@
 <attribute name="VALUE" x="226.06" y="84.074" size="1.778" layer="96" align="bottom-center"/>
 </instance>
-<instance part="R15" gate="G$1" x="180.34" y="55.88">
-<attribute name="NAME" x="180.34" y="57.404" size="1.778" layer="95" font="vector" align="bottom-center"/>
-<attribute name="VALUE" x="180.34" y="54.356" size="1.778" layer="96" font="vector" align="top-center"/>
-</instance>
 <instance part="J1" gate="G$1" x="81.28" y="154.94">
 <attribute name="VALUE" x="76.2" y="145.034" size="1.778" layer="96" font="vector"/>
 <attribute name="NAME" x="76.2" y="165.608" size="1.778" layer="95" font="vector"/>
 </instance>
-<instance part="J2" gate="G$1" x="81.28" y="132.08">
-<attribute name="VALUE" x="76.2" y="122.174" size="1.778" layer="96" font="vector"/>
+<instance part="J2" gate="G$1" x="81.28" y="134.62">
+<attribute name="VALUE" x="76.2" y="127.254" size="1.778" layer="96" font="vector"/>
 <attribute name="NAME" x="76.2" y="142.748" size="1.778" layer="95" font="vector"/>
 </instance>
@@
 <wire x1="190.5" y1="76.2" x2="185.42" y2="76.2" width="0.1524" layer="91"/>
 <wire x1="185.42" y1="76.2" x2="185.42" y2="81.28" width="0.1524" layer="91"/>
-<wire x1="170.18" y1="76.2" x2="185.42" y2="76.2" width="0.1524" layer="91"/>
-<junction x="185.42" y="76.2"/>
-<pinref part="R15" gate="G$1" pin="1"/>
-<wire x1="175.26" y1="55.88" x2="170.18" y2="55.88" width="0.1524" layer="91"/>
-<wire x1="170.18" y1="55.88" x2="170.18" y2="76.2" width="0.1524" layer="91"/>
 </segment>
 <segment>
@@
 <wire x1="86.36" y1="132.08" x2="96.52" y2="132.08" width="0.1524" layer="91"/>
 <label x="91.44" y="132.08" size="1.778" layer="95"/>
-<pinref part="J2" gate="G$1" pin="3"/>
+<pinref part="J2" gate="G$1" pin="1"/>
 </segment>
 </net>
@@
 <wire x1="86.36" y1="134.62" x2="96.52" y2="134.62" width="0.1524" layer="91"/>
 <label x="91.44" y="134.62" size="1.778" layer="95"/>
-<pinref part="J2" gate="G$1" pin="4"/>
+<pinref part="J2" gate="G$1" pin="2"/>
 </segment>
 </net>
@@
 <wire x1="86.36" y1="137.16" x2="96.52" y2="137.16" width="0.1524" layer="91"/>
 <label x="91.44" y="137.16" size="1.778" layer="95"/>
-<pinref part="J2" gate="G$1" pin="5"/>
+<pinref part="J2" gate="G$1" pin="3"/>
 </segment>
 </net>
@@
 <wire x1="86.36" y1="139.7" x2="96.52" y2="139.7" width="0.1524" layer="91"/>
 <label x="91.44" y="139.7" size="1.778" layer="95"/>
-<pinref part="J2" gate="G$1" pin="6"/>
+<pinref part="J2" gate="G$1" pin="4"/>
 </segment>
 </net>
@@
 <label x="228.6" y="104.14" size="1.778" layer="95"/>
 </segment>
-<segment>
-<wire x1="86.36" y1="129.54" x2="96.52" y2="129.54" width="0.1524" layer="91"/>
-<label x="91.44" y="129.54" size="1.778" layer="95"/>
-<pinref part="J2" gate="G$1" pin="2"/>
-</segment>
-</net>
-<net name="SQW" class="0">
-<segment>
-<pinref part="R15" gate="G$1" pin="2"/>
-<pinref part="U2" gate="G$1" pin="INT/SQW"/>
-<wire x1="185.42" y1="55.88" x2="190.5" y2="55.88" width="0.1524" layer="91"/>
-<label x="185.42" y="55.88" size="1.778" layer="95"/>
-</segment>
-<segment>
-<pinref part="J2" gate="G$1" pin="1"/>
-<wire x1="86.36" y1="127" x2="96.52" y2="127" width="0.1524" layer="91"/>
-<label x="91.44" y="127" size="1.778" layer="95"/>
-</segment>
-</net>
+</net>
